File: internal/kicad/testdata/drcboard/board.kicad_pcb (KiCad board)
At the start: 4 copper layers, 4 parts

Commit message: kicad drc / fab --preflight: review fixes (object-level baseline matching, fab warnings gate, rules and contract proofs)
- Baseline matching is by the offending objects: same item-uuid multiset,
  each within tolerance of its baseline position (uuid-less fallback: same
  owners, every item in order within tolerance); warning->error is new.
- --baseline-pcb --out: raw report paths fixed before the parallel runs.
- kicad-drc also gates warning-severity violations of electrical /
  fabrication rules (DRCGatesWarning: hard class + copper_sliver), waivable.
- Preflight parity always uses the project's root schematic from the
  .kicad_pro (else cannot-check); --sch must be a sheet of that hierarchy
  (schematic-root) and the BOM is read from the same root.
- Effective rules: wrong-type values, warning/ignore-severity and min-less
  custom constraints are Unknown (cannot-check); only Board Setup, the
  Default netclass and unconditional error rules prove coverage; zone
  connect_pads clearances count.
- Finish compared as explicit processes (HASL leaded / lead-free, ENIG,
  ENEPIG, OSP, immersion silver / tin, hard gold); ambiguous -> cannot-check.
- Contract sources must name known fields and cover every checked limit,
  the finish and assembly.sides.

Co-Authored-By: Claude Opus 5.5 <noreply@anthropic.com>
Routing:
- net VCC: track 10.0 -> 20.0 mm
Changed lines of the file:
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@@
 	(gr_text "rev A" (at 5 5) (layer "F.SilkS") (uuid "txt-1"))
 	(segment (start 10 10) (end 20 10) (width 0.15) (layer "F.Cu") (net 2) (uuid "trk-1"))
+	(segment (start 10 12) (end 20 12) (width 0.15) (layer "F.Cu") (net 2) (uuid "trk-2"))
 	(arc (start 20 10) (mid 21 11) (end 22 10) (width 0.25) (layer "B.Cu") (net 1) (uuid "arc-1"))
 	(via (at 15 10) (size 0.6) (drill 0.3) (layers "F.Cu" "B.Cu") (net 2) (uuid "via-1"))
